File: schematic_files/DeltaBot.kicad_sch (KiCad schematic)
At the start: 16 parts, among them J1 USB C PD Modulle, J2 LIDAR, J3 MOTOR_L, J4 MOTOR_R, SW1 SW_SPDT, U1 Radxa_ROCK5B, U2 Buck Converter

Commit message: schematic and modified footprints
Parts:
- removed D1, D2: D, deltabot:D_DO-41_SOD81_P10.16mm_Horizontal, symbol Device:D
- removed J2: LIDAR, deltabot:PinHeader_1x07_P2.54mm_Vertical, symbol Connector_Generic:Conn_01x07
- added C7: 5uF, deltabot:C_Disc_D3.0mm_W2.0mm_P2.50mm, symbol Device:C_Polarized
- added J5: C1_LIDAR, Connector_Molex:Molex_KK-254_AE-6410-05A_1x05_P2.54mm_Vertical, symbol Connector:Conn_01x05_Pin
- C3: value 1uF -> 0.1uF
- J1: footprint deltabot:USB_C -> deltabot:USB_PD
Connections:
- net +5V: now also C7.1, J5.1 (VCC)
- net GND: now also C7.2, J5.4 (GND)
- net LIDAR_RX: now also J5.3 (RX)
- net LIDAR_TX: now also J5.2 (TX)
- net MOTO_CTRL: no longer names the net of U1.18 (GPIO4_D4)
- no-connect marks 0 -> 28
Other:
- moved on the sheet: C1, C2, C3, C4, C5, C6, F1, J1, J3, J4, SW1, U1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
