File: schematic_files/deltabot/DeltaBot.kicad_sch (KiCad schematic)
At the start: 15 parts, among them J1 USB C PD Modulle, J3 MOTOR_L, J4 MOTOR_R, J5 C1_LIDAR, SW1 SW_SPDT, U1 Radxa_ROCK5B, U2 Buck Converter

Commit message: pcb v2
Parts:
- removed C3: 0.1uF, Capacitor_SMD:C_0603_1608Metric, symbol Device:C_Polarized
- added C10, C11, C13, C9: 10nF, Capacitor_SMD:C_0805_2012Metric_Pad1.18x1.45mm_HandSolder, symbol Device:C
- added C12, C14, C15, C3, C8: 100nF, Capacitor_SMD:C_0805_2012Metric_Pad1.18x1.45mm_HandSolder, symbol Device:C
- added D1: LED, LED_SMD:LED_0805_2012Metric_Pad1.15x1.40mm_HandSolder, symbol Device:LED
- added IC1: ADS1115LIDGSR, deltabot:SOP50P490X110-10N, symbol ADS1115LIDGSR:ADS1115LIDGSR
- added R1, R2, R3, R5: 10R, Resistor_SMD:R_0805_2012Metric_Pad1.20x1.40mm_HandSolder, symbol Device:R
- added R10, R4, R6, R7, R8: 10k, Resistor_SMD:R_0805_2012Metric_Pad1.20x1.40mm_HandSolder, symbol Device:R
- added R11: 4k7, Resistor_SMD:R_0805_2012Metric_Pad1.20x1.40mm_HandSolder, symbol Device:R
- added R12: 1k, Resistor_SMD:R_0805_2012Metric_Pad1.20x1.40mm_HandSolder, symbol Device:R
- added R9: shunt resistor (wire), Resistor_SMD:R_0805_2012Metric_Pad1.20x1.40mm_HandSolder, symbol Device:R
- C1: footprint Capacitor_THT:CP_Radial_D12.5mm_P5.00mm -> Capacitor_THT:CP_Radial_D16.0mm_P7.50mm
- C2: footprint Capacitor_SMD:C_0603_1608Metric -> Capacitor_SMD:CP_Elec_6.3x3
- C4, C5: value 1uF -> 220uF; footprint Capacitor_SMD:C_0603_1608Metric -> Capacitor_SMD:CP_Elec_6.3x3
- C6: value 1uF -> 10uF; footprint Capacitor_SMD:C_0603_1608Metric -> Capacitor_SMD:CP_Elec_6.3x3
- C7: value 5uF -> 4u7F; footprint Capacitor_SMD:C_0805_2012Metric -> Capacitor_SMD:CP_Elec_6.3x3
Connections:
- net +5V: now also C12.2, C3.1, C8.1, IC1.8 (VDD), R12.1
- net +9V: now also F1.1, R10.1; no longer SW1.1 (A)
- net GND: now also C10.2, C11.2, C12.1, C13.2, C3.2, C8.2, C9.2, D1.2 (A), IC1.3 (GND), R1.2, R11.2, R3.1, R4.1, R9.2; no longer J1.2 (GND)
- net at SW1.2 (B): now also J1.1 (VCC); no longer F1.1
- net at F1.2: now also SW1.1 (A); no longer J1.1 (VCC)
- net +3.3V: now reaches U1.1 (3.3V)
- net +3.3V: now also R6.2, R7.1, R8.1
- net SDA: now reaches U1.3 (I2C7_SDA)
- net SDA: now also IC1.9 (SDA), R8.2
- net ALERT: now reaches U1.38 (GPIO4_A6)
- net ALERT: now also IC1.2 (ALERT/RDY), R6.1
- net ADDR: now reaches U1.40 (GPIO4_A7)
- net ADDR: now also IC1.1 (ADDR), R4.2
- net SCL: now reaches U1.5 (I2C7_SCL)
- net SCL: now also IC1.10 (SCL), R7.2
- new net: C14.1, C9.1, IC1.4 (AIN0), R2.2
- new net: C10.1, C14.2, IC1.5 (AIN1), R3.2
- new net: R10.2, R11.1, R5.2
- new net: C13.1, C15.1, IC1.7 (AIN3), R5.1
- new net: D1.1 (K), R12.2
- new net: C11.1, C15.2, IC1.6 (AIN2), R1.1
- new net shunt: J1.2 (GND_USB), R2.1, R9.1
- no-connect marks 28 -> 23
Other:
- note added: "ADC"
- note added: "LiDAR"
- note added: "Rock 5B+"
- note added: "indicator LED"
- note added: "power distribution"
- note added: "servo motors"
- note removed: "CONNECTORS"
- note removed: "POWER SUPPLY"
- note removed: "ROCK_5B"
- moved on the sheet: C1, C2, C4, C5, C6, C7, F1, J1, J3, J4, SW1, U1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
