File: additional_files/schematic_files/deltabot/DeltaBot.kicad_pcb (KiCad board)
At the start: 2 copper layers, 167.4 x 101.8 mm, 45 parts, among them IC1 ADS1115LIDGSR, J1 USB C PD Modulle, J3 MOTOR_L, J4 MOTOR_R, J5 C1_LIDAR, SW1 SW_SPDT, U1 Radxa_ROCK5B, U2 Buck Converter

Commit message: changes to schematic and pcb
Parts:
- moved R7 3.25 mm to (79.2, 100.8)
- moved C1 2.51 mm to (114.5, 59.2)
Routing:
- net +9V: track 72.5 -> 64.2 mm
- net +5V: track 373.6 -> 380.4 mm
- net GND: track 4.60 -> 0.00 mm
- net +3.3V: track 115.7 -> 112.2 mm
- net PWM_L: track 99.1 -> 101.5 mm
- net SCL: track 41.1 -> 42.9 mm
Other:
- board size 167.4 x 101.8 mm -> 167 x 101.8 mm
