File: additional_files/schematic_files/epsilonbot/DeltaBot.kicad_sch (KiCad schematic)
At the start: 37 parts, among them IC1 ADS1115LIDGSR, J1 USB C PD Modulle, J3 MOTOR_L, J4 MOTOR_R, J5 C1_LIDAR, SW1 SW_SPDT, U1 Radxa_ROCK5B, U2 Buck Converter

Commit message: pcb changes
rerouted to leave more space for the motors, changed clearance width at the request of the rankine technicians, increased width of traces around the ADC
Parts:
- C4, C5: footprint Capacitor_SMD:CP_Elec_6.3x3 -> Capacitor_SMD:CP_Elec_10x10
- C6, C7: footprint Capacitor_SMD:CP_Elec_6.3x3 -> Capacitor_SMD:CP_Elec_6.3x7.7
Connections:
- net ADDR: now also U1.11 (GPIO4_C2); no longer U1.40 (GPIO4_A7)
- net ALERT: now also U1.13 (GPIO4_C6); no longer U1.38 (GPIO4_A6)
Changed lines of the file:
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@@
 	)
 	(no_connect
+		(at 87.63 71.12)
+	)
+	(no_connect
 		(at 26.67 50.8)
 	)
 	(no_connect
-		(at 87.63 50.8)
+		(at 87.63 73.66)
 	)
 	(no_connect
-		(at 87.63 68.58)
+		(at 87.63 50.8)
 	)
 	(no_connect
@@
 	)
 	(no_connect
+		(at 87.63 68.58)
+	)
+	(no_connect
 		(at 26.67 45.72)
 	)
@@
 	)
 	(no_connect
-		(at 26.67 40.64)
-	)
-	(no_connect
-		(at 26.67 38.1)
-	)
-	(no_connect
 		(at 26.67 48.26)
 	)
@@
 	(wire
 		(pts
-			(xy 88.9 71.12) (xy 87.63 71.12)
-		)
-		(stroke
-			(width 0)
-			(type default)
-		)
-	)
-	(wire
-		(pts
 			(xy 220.98 34.29) (xy 233.68 34.29)
 		)
@@
 	(wire
 		(pts
-			(xy 21.59 35.56) (xy 26.67 35.56)
+			(xy 17.78 35.56) (xy 26.67 35.56)
 		)
 		(stroke
@@
 	(wire
 		(pts
-			(xy 21.59 36.83) (xy 21.59 35.56)
+			(xy 17.78 36.83) (xy 17.78 35.56)
 		)
 		(stroke
@@
 	(wire
 		(pts
-			(xy 88.9 73.66) (xy 87.63 73.66)
-		)
-		(stroke
-			(width 0)
-			(type default)
-		)
-	)
-	(wire
-		(pts
 			(xy 137.16 106.68) (xy 137.16 107.95)
 		)
@@
 		)
 	)
+	(global_label "ADDR"
+		(shape input)
+		(at 26.67 38.1 180)
+		(fields_autoplaced yes)
+		(effects
+			(font
+				(size 1.27 1.27)
+			)
+			(justify right)
+		)
+		(property "Intersheetrefs" "${INTERSHEET_REFS}"
+			(at 19.4404 38.1 0)
+			(effects
+				(font
+					(size 1.27 1.27)
+				)
+				(justify right)
+				(hide yes)
+			)
+		)
+	)
 	(global_label "SCL"
 		(shape input)
@@
 	(global_label "ALERT"
 		(shape input)
-		(at 88.9 71.12 0)
+		(at 26.67 40.64 180)
 		(fields_autoplaced yes)
 		(effects
@@
 				(size 1.27 1.27)
 			)
-			(justify left)
+			(justify right)
 		)
 		(property "Intersheetrefs" "${INTERSHEET_REFS}"
-			(at 96.7343 71.12 0)
+			(at 18.8357 40.64 0)
 			(effects
 				(font
 					(size 1.27 1.27)
 				)
-				(justify left)
+				(justify right)
 				(hide yes)
 			)
@@
 		)
 	)
-	(global_label "ADDR"
-		(shape input)
-		(at 88.9 73.66 0)
-		(fields_autoplaced yes)
-		(effects
-			(font
-				(size 1.27 1.27)
-			)
-			(justify left)
-		)
-		(property "Intersheetrefs" "${INTERSHEET_REFS}"
-			(at 96.1296 73.66 0)
-			(effects
-				(font
-					(size 1.27 1.27)
-				)
-				(justify left)
-				(hide yes)
-			)
-		)
-	)
 	(global_label "LIDAR_TX"
 		(shape input)
@@
 	(symbol
 		(lib_id "power:GND")
-		(at 21.59 36.83 0)
+		(at 17.78 36.83 0)
 		(unit 1)
 		(exclude_from_sim no)
@@
 		(dnp no)
 		(property "Reference" "#PWR016"
-			(at 21.59 43.18 0)
+			(at 17.78 43.18 0)
 			(effects
 				(font
@@
 		)
 		(property "Value" "GND"
-			(at 18.796 36.83 0)
+			(at 17.78 33.528 0)
 			(effects
 				(font
@@
 		)
 		(property "Footprint" ""
-			(at 21.59 36.83 0)
+			(at 17.78 36.83 0)
 			(effects
 				(font
@@
 		)
 		(property "Datasheet" ""
-			(at 21.59 36.83 0)
+			(at 17.78 36.83 0)
 			(effects
 				(font
@@
 		)
 		(property "Description" ""
-			(at 21.59 36.83 0)
+			(at 17.78 36.83 0)
 			(effects
 				(font
@@
 			)
 		)
-		(property "Footprint" "Capacitor_SMD:CP_Elec_6.3x3"
+		(property "Footprint" "Capacitor_SMD:CP_Elec_6.3x7.7"
 			(at 215.5952 67.31 0)
 			(effects
@@
 			)
 		)
-		(property "Footprint" "Capacitor_SMD:CP_Elec_6.3x3"
+		(property "Footprint" "Capacitor_SMD:CP_Elec_6.3x7.7"
 			(at 101.2952 27.94 0)
 			(effects
@@
 			)
 		)
-		(property "Footprint" "Capacitor_SMD:CP_Elec_6.3x3"
+		(property "Footprint" "Capacitor_SMD:CP_Elec_10x10"
 			(at 158.4452 66.04 0)
 			(effects
@@
 			)
 		)
-		(property "Footprint" "Capacitor_SMD:CP_Elec_6.3x3"
+		(property "Footprint" "Capacitor_SMD:CP_Elec_10x10"
 			(at 130.5052 66.04 0)
 			(effects

Commit message: removed build
Parts:
- C2: value 1uF -> 10uF
